File: Motorrumsstyrning.kicad_pcb (KiCad board)
At the start: 2 copper layers, 63 x 61 mm, 34 parts, among them IC1 MCP2562-E_P, J1 SD_Card_Connector, J2 Screw_Terminal_01x10, U1 LM1084-5.0, U2 NUCLEO-F303K8

Commit message: Added SD breakout labels and Vera logo on back
Parts:
- added G***: LOGO, Vera-MRS-21:Vera-Logo, B.Cu at (150.0, 77.3)
Other:
- board text added: "Ded"
- board text added: "MISO"
- board text added: "MOSI"
- board text added: "NC"
- board text added: "Tac"
- board text added: "VT-2021 Axel Henriksson Erik Bångsbo"
- board text added: "~CD"
- board text added: "~CS"
- board text added: "~WP"
- board text removed: "26/05/2021 Axel Henriksson Erik Bångsbo"
- board text removed: "De"
- board text removed: "Ta"

Commit message: Added to PCB
Parts:
- removed G***: LOGO, Vera-MRS-21:Vera-Logo
- removed G***: LOGO, Vera-MRS-21:Vera-Logo-Small
- removed IC1: MCP2562-E_P, Vera-MRS-21:DIP781W56P254L950H533Q8N
- removed R4: 50k, Resistor_THT:R_Axial_DIN0204_L3.6mm_D1.6mm_P5.08mm_Horizontal
- removed TP1, TP10, TP11, TP12, TP13, TP14, TP6, TP7, TP8, TP9: TestPoint_Small, TestPoint:TestPoint_Pad_D1.0mm
- added J2: Screw_Terminal_01x10, Vera-MRS-21:TerminalBlock_Phoenix_MPT-0,5-10-2.54_1x10_P2.54mm_Horizontal, F.Cu at (135.0, 121.0)
- added Q1: BC337, Package_TO_SOT_THT:TO-92_Inline, F.Cu at (212.9, 69.5)
- added Q2: BC337, Package_TO_SOT_THT:TO-92_Inline, F.Cu at (195.8, 77.8)
- added R11: R_Small, Resistor_THT:R_Axial_DIN0204_L3.6mm_D1.6mm_P7.62mm_Horizontal, B.Cu at (134.0, 94.0)
- added R8: 1k, Resistor_THT:R_Axial_DIN0204_L3.6mm_D1.6mm_P5.08mm_Horizontal, F.Cu at (193.0, 80.0)
- added U3: MCP2551-I-P, Package_DIP:DIP-8_W7.62mm, F.Cu at (132.4, 91.4)
- J3: renamed from J2; footprint TerminalBlock_Phoenix:TerminalBlock_Phoenix_MPT-0,5-10-2.54_1x10_P2.54mm_Horizontal -> Vera-MRS-21:TerminalBlock_Phoenix_MPT-0,5-10-2.54_1x10_P2.54mm_Horizontal
- U1: moved to B.Cu
- moved U1 49.3 mm to (181.0, 100.0)
- moved R10 10.0 mm to (152.9, 107.8)
- moved R12 10.0 mm to (140.2, 104.1)
- moved R13 10.0 mm to (142.7, 102.9)
- moved R14 10.0 mm to (149.1, 100.2)
- moved R15 10.0 mm to (149.1, 107.8)
- moved U2 10.0 mm to (161.8, 102.7)
- renumbered R9 to R10, R13 to R12, R14 to R13, R10 to R14, R11 to R15, R12 to R16, R8 to R9
Connections:
- J1 pad 1: /~SPI1_CS -> GND
- J3 pad 6: Net-(J2-Pad6) -> /~RST
- U2 pad CN3_1: /USART2_TX -> (no net)
- U2 pad CN3_10: Net-(U2-PadCN3_10) -> /~CD
- U2 pad CN3_11: Net-(U2-PadCN3_11) -> /~WP
- U2 pad CN3_12: Net-(U2-PadCN3_12) -> /PA8
- U2 pad CN3_14: Net-(U2-PadCN3_14) -> /PB5
- U2 pad CN3_15: Net-(U2-PadCN3_15) -> /PB4
- U2 pad CN3_2: /USAR2_RX -> (no net)
- U2 pad CN3_3: Net-(U2-PadCN3_3) -> /~RST
- U2 pad CN3_4: Net-(U2-PadCN3_4) -> GND
- U2 pad CN3_6: Net-(U2-PadCN3_6) -> /PB0
- U2 pad CN3_9: Net-(U2-PadCN3_9) -> /PB1
- U2 pad CN4_10: Net-(U2-PadCN4_10) -> /Injector_Enable
- U2 pad CN4_13: Net-(U2-PadCN4_13) -> (no net)
- U2 pad CN4_15: Net-(U2-PadCN4_15) -> /PB3
- U2 pad CN4_2: Net-(U2-PadCN4_2) -> GND
- U2 pad CN4_3: Net-(U2-PadCN4_3) -> /~RST
- U2 pad CN4_5: Net-(U2-PadCN4_5) -> /Start_Enable
- U2 pad CN4_9: Net-(U2-PadCN4_9) -> /PA4
Other:
- board size 63 x 61 mm -> 74.8 x 61 mm
- board text added: "Dead"
- board text added: "StrtR"
- board text added: "Tach"
- board text added: "~RST"
- board text removed: "Ded"
- board text removed: "SR"
- board text removed: "Tac"

Commit message: First complete draft
Parts:
- removed the Q1 at (212.9, 69.5)
- added G***: LOGO, Vera-MRS-21:Vera-Logo-Small, F.Cu at (172.7, 88.3)
- added J10: Jumper, Vera-MRS-21:THT_Jumper, F.Cu at (139.7, 113.0)
- added J11: Jumper, Vera-MRS-21:THT_Jumper, F.Cu at (133.3, 74.3)
- added J12: Jumper, Vera-MRS-21:THT_Jumper, F.Cu at (133.0, 80.6)
- added J13: Jumper, Vera-MRS-21:THT_Jumper, F.Cu at (133.3, 76.8)
- added J14: Jumper, Vera-MRS-21:THT_Jumper, F.Cu at (144.8, 114.9)
- added J15: Jumper, Vera-MRS-21:THT_Jumper, F.Cu at (147.3, 114.9)
- added J16: Jumper, Vera-MRS-21:THT_Jumper, F.Cu at (149.9, 114.9)
- added J17: Jumper, Vera-MRS-21:THT_Jumper, F.Cu at (152.4, 114.9)
- added J18: Jumper, Vera-MRS-21:THT_Jumper, F.Cu at (154.9, 114.9)
- added J19: Jumper, Vera-MRS-21:THT_Jumper, F.Cu at (157.5, 114.9)
- added J20: Jumper, Vera-MRS-21:THT_Jumper, F.Cu at (160.0, 114.9)
- added J21: Jumper, Vera-MRS-21:THT_Jumper, F.Cu at (162.6, 114.9)
- added J22: Jumper, Vera-MRS-21:THT_Jumper, F.Cu at (142.2, 113.0)
- added J23: Screw_Terminal_01x10, Vera-MRS-21:TerminalBlock_Phoenix_MPT-0,5-10-2.54_1x10_P2.54mm_Horizontal, F.Cu at (144.8, 120.0)
- added J3: Jumper, Vera-MRS-21:THT_Jumper, F.Cu at (149.9, 91.4)
- added J4: Jumper, Vera-MRS-21:THT_Jumper, F.Cu at (157.5, 91.4)
- added J5: Jumper, Vera-MRS-21:THT_Jumper, F.Cu at (160.0, 91.4)
- added J6: Jumper, Vera-MRS-21:THT_Jumper, F.Cu at (142.2, 91.4)
- added J7: Jumper, Vera-MRS-21:THT_Jumper, F.Cu at (144.8, 91.4)
- added J8: Jumper, Vera-MRS-21:THT_Jumper, F.Cu at (152.4, 91.4)
- added J9: Jumper, Vera-MRS-21:THT_Jumper, F.Cu at (154.9, 91.4)
- added JP1: CS_Jumper, Jumper:SolderJumper-2_P1.3mm_Open_TrianglePad1.0x1.5mm, F.Cu at (130.6, 94.6)
- added JP2: SolderJumper_2_Bridged, Jumper:SolderJumper-2_P1.3mm_Bridged2Bar_RoundedPad1.0x1.5mm, B.Cu at (144.8, 112.4)
- added JP3: SolderJumper_2_Bridged, Jumper:SolderJumper-2_P1.3mm_Bridged2Bar_RoundedPad1.0x1.5mm, B.Cu at (147.3, 112.4)
- added JP4: SolderJumper_2_Bridged, Jumper:SolderJumper-2_P1.3mm_Bridged2Bar_RoundedPad1.0x1.5mm, B.Cu at (149.9, 112.4)
- added JP5: SolderJumper_2_Bridged, Jumper:SolderJumper-2_P1.3mm_Bridged2Bar_RoundedPad1.0x1.5mm, B.Cu at (152.4, 112.4)
- added JP6: SolderJumper_2_Bridged, Jumper:SolderJumper-2_P1.3mm_Bridged2Bar_RoundedPad1.0x1.5mm, B.Cu at (154.9, 112.4)
- added JP7: SolderJumper_2_Bridged, Jumper:SolderJumper-2_P1.3mm_Bridged2Bar_RoundedPad1.0x1.5mm, B.Cu at (157.5, 112.4)
- added JP8: SolderJumper_2_Bridged, Jumper:SolderJumper-2_P1.3mm_Bridged2Bar_RoundedPad1.0x1.5mm, B.Cu at (160.0, 112.4)
- added JP9: SolderJumper_2_Bridged, Jumper:SolderJumper-2_P1.3mm_Bridged2Bar_RoundedPad1.0x1.5mm, B.Cu at (162.6, 112.4)
- added Q2: BC337, Package_TO_SOT_THT:TO-92_Inline, F.Cu at (165.1, 114.3)
- added R4: 50k, Resistor_THT:R_Axial_DIN0207_L6.3mm_D2.5mm_P7.62mm_Horizontal, B.Cu at (139.1, 99.1)
- J2: value Screw_Terminal_01x10 -> Jumper; footprint Vera-MRS-21:TerminalBlock_Phoenix_MPT-0,5-10-2.54_1x10_P2.54mm_Horizontal -> Vera-MRS-21:THT_Jumper
- R1, R2, R3, R5, R6, R7: footprint Resistor_THT:R_Axial_DIN0204_L3.6mm_D1.6mm_P5.08mm_Horizontal -> Resistor_THT:R_Axial_DIN0207_L6.3mm_D2.5mm_P7.62mm_Horizontal; moved to B.Cu
- R10: value 10k -> 1k; footprint Resistor_THT:R_Axial_DIN0204_L3.6mm_D1.6mm_P5.08mm_Horizontal -> Resistor_THT:R_Axial_DIN0207_L6.3mm_D2.5mm_P7.62mm_Horizontal
- R11: value R_Small -> 1k; footprint Resistor_THT:R_Axial_DIN0204_L3.6mm_D1.6mm_P7.62mm_Horizontal -> Resistor_THT:R_Axial_DIN0207_L6.3mm_D2.5mm_P7.62mm_Horizontal
- R12: value 1k -> 4k2; footprint Resistor_THT:R_Axial_DIN0204_L3.6mm_D1.6mm_P5.08mm_Horizontal -> Resistor_THT:R_Axial_DIN0207_L6.3mm_D2.5mm_P7.62mm_Horizontal
- R13: value 1k -> 10k; footprint Resistor_THT:R_Axial_DIN0204_L3.6mm_D1.6mm_P5.08mm_Horizontal -> Resistor_THT:R_Axial_DIN0207_L6.3mm_D2.5mm_P7.62mm_Horizontal
- R14: value 4k2 -> 1k; footprint Resistor_THT:R_Axial_DIN0204_L3.6mm_D1.6mm_P5.08mm_Horizontal -> Resistor_THT:R_Axial_DIN0207_L6.3mm_D2.5mm_P7.62mm_Horizontal; moved to F.Cu
- R15: value 10k -> R_Small; footprint Resistor_THT:R_Axial_DIN0204_L3.6mm_D1.6mm_P5.08mm_Horizontal -> Resistor_THT:R_Axial_DIN0207_L6.3mm_D2.5mm_P7.62mm_Horizontal
- R16: footprint Resistor_THT:R_Axial_DIN0204_L3.6mm_D1.6mm_P5.08mm_Horizontal -> Resistor_THT:R_Axial_DIN0207_L6.3mm_D2.5mm_P7.62mm_Horizontal; moved to F.Cu
- R8: value 1k -> 4k2; footprint Resistor_THT:R_Axial_DIN0204_L3.6mm_D1.6mm_P5.08mm_Horizontal -> Resistor_THT:R_Axial_DIN0207_L6.3mm_D2.5mm_P7.62mm_Horizontal; moved to B.Cu
- R9: value 4k2 -> 10k; footprint Resistor_THT:R_Axial_DIN0204_L3.6mm_D1.6mm_P5.08mm_Horizontal -> Resistor_THT:R_Axial_DIN0207_L6.3mm_D2.5mm_P7.62mm_Horizontal
- U1: value LM1084-5.0 -> NUCLEO-F303K8; footprint Package_TO_SOT_THT:TO-220-3_Horizontal_TabDown -> Vera-MRS-21:NUCLEO_32; moved to F.Cu
- U2: value NUCLEO-F303K8 -> LM1084-5.0; footprint Vera-MRS-21:NUCLEO_32 -> Package_TO_SOT_THT:TO-220-3_Horizontal_TabDown; moved to B.Cu
- moved Q1 72.3 mm to (127.5, 101.6)
- moved R8 54.2 mm to (145.4, 106.0)
- moved R3 41.2 mm to (170.8, 106.0), turned to 90 degrees
- moved R2 36.5 mm to (134.6, 94.6), turned to 180 degrees
- moved U2 34.5 mm to (135.3, 80.6), turned to 90 degrees
- moved R11 32.8 mm to (164.5, 106.0), turned to 90 degrees
- moved J2 32.0 mm to (147.3, 91.4)
- moved R15 30.1 mm to (130.8, 83.8), turned to 270 degrees
- moved R1 20.7 mm to (161.3, 106.0), turned to 90 degrees
- moved U1 19.5 mm to (161.6, 102.2)
- moved R5 16.5 mm to (142.2, 106.0), turned to 90 degrees
- moved R14 15.8 mm to (134.0, 104.8), turned to 90 degrees
- moved R6 15.7 mm to (158.1, 106.0), turned to 90 degrees
- moved R10 14.9 mm to (167.6, 106.0), turned to 90 degrees
- moved R13 13.0 mm to (154.9, 98.4), turned to 270 degrees
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- renumbered J3 to J24, Q2 to Q1
Connections:
- J1 pad 1: GND -> /~CS
- J2 pad 1: /PB0 -> GND
- J24 pad 4: /I2C1_SDA -> /I2C1_SCL
- J24 pad 5: /I2C1_SCL -> /I2C1_SDA
- Q1 pad 2: Net-(Q2-Pad2) -> Net-(Q1-Pad2)
- R10 pad 1: /Tachometer -> +3V3
- R10 pad 2: GND -> /I2C1_SDA
- R11 pad 1: GND -> +3V3
- R11 pad 2: Net-(R11-Pad2) -> /I2C1_SCL
- R12 pad 1: +3V3 -> /Deadmans_12V
- R12 pad 2: /I2C1_SCL -> /Deadmans
- R13 pad 1: +3V3 -> /Deadmans
- R13 pad 2: /I2C1_SDA -> GND
- R14 pad 1: /Deadmans_12V -> Net-(Q1-Pad2)
- R14 pad 2: /Deadmans -> /Start_Enable
- R15 pad 1: /Deadmans -> GND
- R15 pad 2: GND -> Net-(R15-Pad2)
- R2 pad 1: +3V3 -> /~CS
- R2 pad 2: /~WP -> GND
- R3 pad 2: Net-(J1-Pad9) -> /~WP
- R8 pad 1: Net-(Q2-Pad2) -> /Tach_12V
- R8 pad 2: /Start_Enable -> /Tachometer
- R9 pad 1: /Tach_12V -> /Tachometer
- R9 pad 2: /Tachometer -> GND
- U3 pad 5: (no net) -> Net-(U3-Pad5)
- U3 pad 8: Net-(R11-Pad2) -> Net-(R15-Pad2)
Routing:
- net +5V: track 0.00 -> 74.9 mm
- net /~RST: track 0.00 -> 70.9 mm
- net /I2C1_SDA: track 0.00 -> 59.1 mm
- net /I2C1_SCL: track 0.00 -> 55.3 mm
- net /SPI1_MOSI: track 0.00 -> 45.0 mm, vias 0 -> 1
- net /CAN_TX: track 0.00 -> 34.3 mm
- net /Deadmans_12V: track 0.00 -> 33.9 mm
- net /USART2_TX: track 0.00 -> 32.0 mm, vias 0 -> 1
- net /USART2_RX: track 0.00 -> 30.8 mm, vias 0 -> 1
- net /Tach_12V: track 0.00 -> 28.5 mm
- net /SPI1_SCK: track 0.00 -> 26.7 mm
- net /SPI1_MISO: track 0.00 -> 25.9 mm
- net +12V: track 0.00 -> 24.3 mm
- net /CAN_RX: track 0.00 -> 24.0 mm
- net /PA8: track 0.00 -> 18.2 mm
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- added copper zone on In2.Cu, net +3V3
- added copper zone on In1.Cu, net GND
- added copper zone on In2.Cu, net GND
Other:
- board size 74.8 x 61 mm -> 65 x 60.5 mm
- copper layers 2 -> 4
- board text added: "+3V3"
- board text added: "12V"
- board text added: "5V"
- board text added: "A0"
- board text added: "A1"
- board text added: "A3"
- board text added: "A4"
- board text added: "AR"
- board text added: "ARF"
- board text added: "B3"
- board text added: "CS_JP"
- board text added: "IN"
- board text added: "OUT"
- board text added: "PA0"
- board text added: "PA1"
- board text added: "PA3"
- board text added: "PA4"
- board text added: "PB3"
- board text added: "RX"
- board text added: "Rev. A Axel Henriksson Erik Bångsbo"
- board text added: "SCK"
- board text added: "SD Breakout"
- board text added: "TX"
- board text removed: "NC"
- board text removed: "Rev. A Vera-MRS-21"
- board text removed: "VT-2021 Axel Henriksson Erik Bångsbo"
