File: Motorrumsstyrning.kicad_pcb (KiCad board)
At the start: 4 copper layers, 65 x 60.5 mm, 54 parts, among them J1 Jumper, J10 Jumper, J11 Jumper, J12 SD_Card_Connector, J13 Jumper, J14 Conn_01x09, J15 Screw_Terminal_01x10, J2 Jumper, J3 Jumper, J4 Jumper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

Commit message: Update
Other:
- rule solder_mask_min_width: 0.25 -> 0.2
Changed lines of the file:
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@@
     (pad_drill 0.762)
     (pad_to_mask_clearance 0.051)
-    (solder_mask_min_width 0.25)
+    (solder_mask_min_width 0.2)
     (aux_axis_origin 0 0)
     (visible_elements 7FFFFFFF)
