File: Motorrumsstyrning.sch (KiCad schematic (older format))
At the start: 35 parts, among them IC1 MCP2562-E_P, J1 SD_Card_Connector, J2 Screw_Terminal_01x10, U1 LM1084-5.0, U2 NUCLEO-F303K8

Commit message: Recommit
Parts:
- gave numbers to parts that had none: 2
Changed lines of the file:
@@
 CANL
 $Comp
-L power:+3V3 #PWR?
+L power:+3V3 #PWR0101
 U 1 1 60B4D1BC
 P 10200 4700
-F 0 "#PWR?" H 10200 4550 50  0001 C CNN
+F 0 "#PWR0101" H 10200 4550 50  0001 C CNN
 F 1 "+3V3" H 10215 4873 50  0000 C CNN
 F 2 "" H 10200 4700 50  0001 C CNN
@@
 $EndComp
 $Comp
-L Device:R_Small R?
+L Device:R_Small R14
 U 1 1 60B4D89B
 P 10300 4850
-F 0 "R?" H 10359 4896 50  0000 L CNN
+F 0 "R14" H 10359 4896 50  0000 L CNN
 F 1 "1k" H 10359 4805 50  0000 L CNN
 F 2 "Resistor_THT:R_Axial_DIN0204_L3.6mm_D1.6mm_P5.08mm_Horizontal" H 10300 4850 50  0001 C CNN
@@
 Connection ~ 10600 5050
 $Comp
-L Device:R_Small R?
+L Device:R_Small R13
 U 1 1 60B53DE1
 P 10100 4850
-F 0 "R?" H 10159 4896 50  0000 L CNN
+F 0 "R13" H 10159 4896 50  0000 L CNN
 F 1 "1k" H 10159 4805 50  0000 L CNN
 F 2 "Resistor_THT:R_Axial_DIN0204_L3.6mm_D1.6mm_P5.08mm_Horizontal" H 10100 4850 50  0001 C CNN

Commit message: Moved terminal block, Added Testpoint labels
Other:
- moved on the sheet: R13, R14
Changed lines of the file:
@@
 Text Notes 500  1300 0    50   ~ 0
 7. Se om Test Points behövs eller om skruvarna fyller samma funktion.
-Text Label 9700 5050 0    50   ~ 0
+Text Label 9450 5250 0    50   ~ 0
 I2C1_SDA
-Text Label 9700 5150 0    50   ~ 0
+Text Label 9450 5350 0    50   ~ 0
 I2C1_SCL
 Text Label 9900 5550 0    50   ~ 0
 Start_Relay_GND
-Text Label 10300 5250 0    50   ~ 0
+Text Label 10300 5150 0    50   ~ 0
 CANH
-Text Label 10300 5350 0    50   ~ 0
+Text Label 10300 5050 0    50   ~ 0
 CANL
 $Comp
 L power:+3V3 #PWR0101
 U 1 1 60B4D1BC
-P 10200 4700
-F 0 "#PWR0101" H 10200 4550 50  0001 C CNN
-F 1 "+3V3" H 10215 4873 50  0000 C CNN
-F 2 "" H 10200 4700 50  0001 C CNN
-F 3 "" H 10200 4700 50  0001 C CNN
-	1    10200 4700
+P 9950 4900
+F 0 "#PWR0101" H 9950 4750 50  0001 C CNN
+F 1 "+3V3" H 9965 5073 50  0000 C CNN
+F 2 "" H 9950 4900 50  0001 C CNN
+F 3 "" H 9950 4900 50  0001 C CNN
+	1    9950 4900
 	1    0    0    -1
 $EndComp
@@
 L Device:R_Small R14
 U 1 1 60B4D89B
-P 10300 4850
-F 0 "R14" H 10359 4896 50  0000 L CNN
-F 1 "1k" H 10359 4805 50  0000 L CNN
-F 2 "Resistor_THT:R_Axial_DIN0204_L3.6mm_D1.6mm_P5.08mm_Horizontal" H 10300 4850 50  0001 C CNN
-F 3 "~" H 10300 4850 50  0001 C CNN
-	1    10300 4850
+P 10000 5050
+F 0 "R14" H 10059 5096 50  0000 L CNN
+F 1 "1k" H 10059 5005 50  0000 L CNN
+F 2 "Resistor_THT:R_Axial_DIN0204_L3.6mm_D1.6mm_P5.08mm_Horizontal" H 10000 5050 50  0001 C CNN
+F 3 "~" H 10000 5050 50  0001 C CNN
+	1    10000 5050
 	1    0    0    -1
 $EndComp
 Wire Wire Line
-	10600 5050 10300 5050
-Wire Wire Line
-	10300 5050 10300 4950
-Connection ~ 10600 5050
+	10000 5250 10000 5150
 $Comp
 L Device:R_Small R13
 U 1 1 60B53DE1
-P 10100 4850
-F 0 "R13" H 10159 4896 50  0000 L CNN
-F 1 "1k" H 10159 4805 50  0000 L CNN
-F 2 "Resistor_THT:R_Axial_DIN0204_L3.6mm_D1.6mm_P5.08mm_Horizontal" H 10100 4850 50  0001 C CNN
-F 3 "~" H 10100 4850 50  0001 C CNN
-	1    10100 4850
-	1    0    0    -1
+P 9900 5050
+F 0 "R13" H 9959 5096 50  0000 L CNN
+F 1 "1k" H 9959 5005 50  0000 L CNN
+F 2 "Resistor_THT:R_Axial_DIN0204_L3.6mm_D1.6mm_P5.08mm_Horizontal" H 9900 5050 50  0001 C CNN
+F 3 "~" H 9900 5050 50  0001 C CNN
+	1    9900 5050
+	-1   0    0    -1
 $EndComp
 Wire Wire Line
-	10600 5150 10100 5150
+	9900 5350 9900 5150
 Wire Wire Line
-	10100 5150 10100 4950
-Connection ~ 10600 5150
+	9900 4950 9950 4950
 Wire Wire Line
-	10300 5050 9700 5050
-Connection ~ 10300 5050
+	10300 5150 10600 5150
 Wire Wire Line
-	9700 5150 10100 5150
-Connection ~ 10100 5150
-Wire Wire Line
-	10100 4750 10200 4750
-Wire Wire Line
-	10200 4750 10200 4700
-Connection ~ 10200 4750
-Wire Wire Line
-	10200 4750 10300 4750
-Wire Wire Line
-	10300 5250 10600 5250
-Connection ~ 10600 5250
-Wire Wire Line
-	10300 5350 10600 5350
-Connection ~ 10600 5350
+	10300 5050 10600 5050
 Wire Wire Line
 	9900 5550 10600 5550
@@
 Text Notes 500  1400 0    50   ~ 0
 8. Göra plats för det elektromagnetiska frihjulet
+Connection ~ 10600 5250
+Connection ~ 10600 5350
+Connection ~ 10600 5050
+Connection ~ 10600 5150
+Wire Wire Line
+	9950 4900 9950 4950
+Connection ~ 9950 4950
+Wire Wire Line
+	9950 4950 10000 4950
+Connection ~ 9900 5350
+Wire Wire Line
+	9900 5350 10600 5350
+Connection ~ 10000 5250
+Wire Wire Line
+	10000 5250 10600 5250
+Wire Wire Line
+	9450 5350 9900 5350
+Wire Wire Line
+	9450 5250 10000 5250
 $EndSCHEMATC

Commit message: CAN tranciever o transistor
Parts:
- removed IC1: MCP2562-E_P, Vera-MRS-21:DIP781W56P254L950H533Q8N, symbol Vera-MRS-21:MCP2562-E_P
- added J?: Screw_Terminal_01x10, TerminalBlock_Phoenix:TerminalBlock_Phoenix_MPT-0,5-10-2.54_1x10_P2.54mm_Horizontal, symbol Motorrumsstyrning-rescue:Screw_Terminal_01x10-Connector
- added Q? (x2): BC337, Package_TO_SOT_THT:TO-92_Inline, symbol Transistor_BJT:BC337
- added R?: R_Small, symbol Device:R_Small
- added R?: 1k, symbol Device:R_Small
- added U?: MCP2551-I-P, Package_DIP:DIP-8_W7.62mm, symbol Interface_CAN_LIN:MCP2551-I-P
- C1, C2: symbol Device:C_Small -> Motorrumsstyrning-rescue:C_Small-Device
- H1, H2, H3, H4: symbol Mechanical:MountingHole_Pad -> Motorrumsstyrning-rescue:MountingHole_Pad-Mechanical
- J2: symbol Connector:Screw_Terminal_01x10 -> Motorrumsstyrning-rescue:Screw_Terminal_01x10-Connector
- R1, R10, R11, R12, R13, R14, R2, R3, R4, R5, R6, R7, R8, R9: symbol Device:R_Small -> Motorrumsstyrning-rescue:R_Small-Device
- TP1, TP10, TP11, TP12, TP13, TP14, TP6, TP7, TP8, TP9: symbol Connector:TestPoint_Small -> Motorrumsstyrning-rescue:TestPoint_Small-Connector
- U1: symbol Regulator_Linear:LM1084-5.0 -> Motorrumsstyrning-rescue:LM1084-5.0-Regulator_Linear
Connections:
- net labels added: Injector_Enable, Injector_IN, Injector_OUT, Start_Enable
- wire segments 87 -> 94
Other:
- note added: "Kolla om 1k gäller för 3.3V vid gate"

Commit message: Added programing folder
Connections:
- net labels added: PA4, PA8, PB0, PB1, PB3, PB4, PB5, PF0, PF1
- wire segments 94 -> 101
Changed lines of the file:
@@
 EESchema Schematic File Version 4
-EELAYER 30 0
+LIBS:Motorrumsstyrning-cache
+EELAYER 29 0
 EELAYER END
 $Descr A4 11693 8268
@@
 L Motorrumsstyrning-rescue:+5V-power #PWR013
 U 1 1 60B01412
-P 9800 950
-F 0 "#PWR013" H 9800 800 50  0001 C CNN
-F 1 "+5V" H 9815 1123 50  0000 C CNN
-F 2 "" H 9800 950 50  0001 C CNN
-F 3 "" H 9800 950 50  0001 C CNN
-	1    9800 950
+P 9900 1100
+F 0 "#PWR013" H 9900 950 50  0001 C CNN
+F 1 "+5V" H 9915 1273 50  0000 C CNN
+F 2 "" H 9900 1100 50  0001 C CNN
+F 3 "" H 9900 1100 50  0001 C CNN
+	1    9900 1100
 	1    0    0    -1
 $EndComp
@@
 U 1 1 60C52B5A
 P 9900 1500
-F 0 "U?" H 10150 2100 50  0000 C CNN
-F 1 "MCP2551-I-P" H 10200 2000 50  0000 C CNN
+F 0 "U?" H 10250 1850 50  0000 C CNN
+F 1 "MCP2551-I-P" H 9500 1850 50  0000 C CNN
 F 2 "Package_DIP:DIP-8_W7.62mm" H 9900 1000 50  0001 C CIN
 F 3 "http://ww1.microchip.com/downloads/en/devicedoc/21667d.pdf" H 9900 1500 50  0001 C CNN
@@
 	1    0    0    -1
 $EndComp
-Wire Wire Line
-	9800 950  9800 1100
-Wire Wire Line
-	9800 1100 9900 1100
 $Comp
 L Device:R_Small R?
@@
 Wire Wire Line
 	6950 2000 8000 2000
+Text Label 5450 3650 0    50   ~ 0
+PB0
+Text Label 5450 3750 0    50   ~ 0
+PB1
+Text Label 5450 3950 0    50   ~ 0
+PB3
+Text Label 5450 4050 0    50   ~ 0
+PB4
+Text Label 5450 4150 0    50   ~ 0
+PB5
+Text Label 5250 4500 0    50   ~ 0
+PF0
+Text Label 5250 4600 0    50   ~ 0
+PF1
+Text Label 6950 3950 2    50   ~ 0
+PA4
+Wire Wire Line
+	6800 3950 6950 3950
+Wire Wire Line
+	5600 3650 5450 3650
+Wire Wire Line
+	5600 3750 5450 3750
+Wire Wire Line
+	5600 3950 5450 3950
+Wire Wire Line
+	5450 4050 5600 4050
+Wire Wire Line
+	5450 4150 5600 4150
+Text Label 6950 4350 2    50   ~ 0
+PA8
+Wire Wire Line
+	6950 4350 6800 4350
+Wire Wire Line
+	5600 4500 5250 4500
+Wire Wire Line
+	5600 4600 5250 4600
 $EndSCHEMATC

Commit message: Added to PCB
Parts:
- removed R4: 50k, Resistor_THT:R_Axial_DIN0204_L3.6mm_D1.6mm_P5.08mm_Horizontal, symbol Motorrumsstyrning-rescue:R_Small-Device
- removed TP1, TP10, TP11, TP12, TP13, TP14, TP6, TP7, TP8, TP9: TestPoint_Small, TestPoint:TestPoint_Pad_D1.0mm, symbol Motorrumsstyrning-rescue:TestPoint_Small-Connector
- J2: renamed from J?; footprint TerminalBlock_Phoenix:TerminalBlock_Phoenix_MPT-0,5-10-2.54_1x10_P2.54mm_Horizontal -> Vera-MRS-21:TerminalBlock_Phoenix_MPT-0,5-10-2.54_1x10_P2.54mm_Horizontal
- J3: renamed from J2; footprint TerminalBlock_Phoenix:TerminalBlock_Phoenix_MPT-0,5-10-2.54_1x10_P2.54mm_Horizontal -> Vera-MRS-21:TerminalBlock_Phoenix_MPT-0,5-10-2.54_1x10_P2.54mm_Horizontal
- R11: renamed from R?; footprint (none) -> Resistor_THT:R_Axial_DIN0204_L3.6mm_D1.6mm_P7.62mm_Horizontal
- R8: renamed from R?; footprint (none) -> Resistor_THT:R_Axial_DIN0204_L3.6mm_D1.6mm_P5.08mm_Horizontal
- gave numbers to parts that had none: 3
- renumbered R9 to R10, R13 to R12, R14 to R13, R10 to R14, R11 to R15, R12 to R16, R8 to R9
Connections:
- net labels added: PB2, ~RST
- net labels removed: PF0, PF1, ~SPI1_CS
Other:
- note added: "6. Kolla vad VREF ska vara på STM32 och CAN transceiver"
- note added: "Left Screw Terminal"
- note added: "Right Screw Terminal"
- note added: "Transistors"
- note removed: "3. Se över ordning och antal i terminalblocket."
- note removed: "4. Se över Deadman_Signal kontra Deadmans_Button"
- note removed: "6. Filtrera och begränsa +12V om VIN är kopplad till den."
- note removed: "7. Se om Test Points behövs eller om skruvarna fyller samma funktion."
- note removed: "8. Göra plats för det elektromagnetiska frihjulet"
- note removed: "Kolla om 1k gäller för 3.3V vid gate"
- note removed: "Screw Terminal"
- moved on the sheet: J2, Q1, Q2, R5, R6, R7, R8, U2

Commit message: First complete draft
Parts:
- added J10, J11, J12, J13, J14, J15, J16, J17, J18, J19, J2, J20, J21, J22, J3, J4, J5, J6, J7, J8, J9: Jumper, Vera-MRS-21:THT_Jumper, symbol Connector:Conn_01x01_Female
- added JP1: CS_Jumper, Jumper:SolderJumper-2_P1.3mm_Open_TrianglePad1.0x1.5mm, symbol Jumper:SolderJumper_2_Open
- added JP2, JP3, JP4, JP5, JP6, JP7, JP8, JP9: SolderJumper_2_Bridged, Jumper:SolderJumper-2_P1.3mm_Bridged2Bar_RoundedPad1.0x1.5mm, symbol Jumper:SolderJumper_2_Bridged
- added R2: 50k, Resistor_THT:R_Axial_DIN0207_L6.3mm_D2.5mm_P7.62mm_Horizontal, symbol Motorrumsstyrning-rescue:R_Small-Device
- R1, R16, R5, R6, R7: footprint Resistor_THT:R_Axial_DIN0204_L3.6mm_D1.6mm_P5.08mm_Horizontal -> Resistor_THT:R_Axial_DIN0207_L6.3mm_D2.5mm_P7.62mm_Horizontal
- R10: renamed from R12; footprint Resistor_THT:R_Axial_DIN0204_L3.6mm_D1.6mm_P5.08mm_Horizontal -> Resistor_THT:R_Axial_DIN0207_L6.3mm_D2.5mm_P7.62mm_Horizontal
- R11: renamed from R13; footprint Resistor_THT:R_Axial_DIN0204_L3.6mm_D1.6mm_P5.08mm_Horizontal -> Resistor_THT:R_Axial_DIN0207_L6.3mm_D2.5mm_P7.62mm_Horizontal
- R12: renamed from R14; footprint Resistor_THT:R_Axial_DIN0204_L3.6mm_D1.6mm_P5.08mm_Horizontal -> Resistor_THT:R_Axial_DIN0207_L6.3mm_D2.5mm_P7.62mm_Horizontal
- R13: renamed from R15; footprint Resistor_THT:R_Axial_DIN0204_L3.6mm_D1.6mm_P5.08mm_Horizontal -> Resistor_THT:R_Axial_DIN0207_L6.3mm_D2.5mm_P7.62mm_Horizontal
- R14: renamed from R8; footprint Resistor_THT:R_Axial_DIN0204_L3.6mm_D1.6mm_P5.08mm_Horizontal -> Resistor_THT:R_Axial_DIN0207_L6.3mm_D2.5mm_P7.62mm_Horizontal
- R15: renamed from R11; footprint Resistor_THT:R_Axial_DIN0204_L3.6mm_D1.6mm_P7.62mm_Horizontal -> Resistor_THT:R_Axial_DIN0207_L6.3mm_D2.5mm_P7.62mm_Horizontal
- R3: renamed from R2; footprint Resistor_THT:R_Axial_DIN0204_L3.6mm_D1.6mm_P5.08mm_Horizontal -> Resistor_THT:R_Axial_DIN0207_L6.3mm_D2.5mm_P7.62mm_Horizontal
- R4: renamed from R3; footprint Resistor_THT:R_Axial_DIN0204_L3.6mm_D1.6mm_P5.08mm_Horizontal -> Resistor_THT:R_Axial_DIN0207_L6.3mm_D2.5mm_P7.62mm_Horizontal
- R8: renamed from R9; footprint Resistor_THT:R_Axial_DIN0204_L3.6mm_D1.6mm_P5.08mm_Horizontal -> Resistor_THT:R_Axial_DIN0207_L6.3mm_D2.5mm_P7.62mm_Horizontal
- R9: renamed from R10; footprint Resistor_THT:R_Axial_DIN0204_L3.6mm_D1.6mm_P5.08mm_Horizontal -> Resistor_THT:R_Axial_DIN0207_L6.3mm_D2.5mm_P7.62mm_Horizontal
- renumbered J2 to J23, J3 to J24, Q2 to Q1, Q1 to Q2, U2 to U1, U1 to U2
Connections:
- net +12V: now also J11.1 (Pin_1); no longer U1.CN4_1 (VIN)
- net +3V3: now also J3.1 (Pin_1)
- net +5V: now also J13.1 (Pin_1)
- net Deadmans: now also U1.CN3_10 (PF0); no longer U1.CN4_12 (PA0)
- net GND: now also J12.1 (Pin_1), J2.1 (Pin_1), J22.1 (Pin_1), R2.2; no longer J1.1 (DAT3/~CS)
- net I2C1_SCL: now also J24.4 (Pin_4), R11.2; no longer J24.5 (Pin_5), R10.2
- net I2C1_SDA: now also J24.5 (Pin_5), R10.2; no longer J24.4 (Pin_4), R11.2
- net Injector_Enable: now also U1.CN4_5 (PA2); no longer U1.CN4_10 (PA3)
- net PA4: now also JP7.1 (A); no longer J23.7 (Pin_7)
- net PA8: now also JP3.1 (A); no longer J23.8 (Pin_8)
- net PB3: now also JP2.1 (A); no longer J23.4 (Pin_4)
- net PB4: now also JP1.2 (B); no longer J23.5 (Pin_5)
- net SPI1_MISO: now also J9.1 (Pin_1)
- net SPI1_MOSI: now also J7.1 (Pin_1)
- net SPI1_SCK: now also J8.1 (Pin_1)
- net Start_Enable: now also U1.CN3_14 (PB5); no longer U1.CN4_5 (PA2)
- net Tachometer: now also U1.CN3_11 (PF1); no longer U1.CN4_11 (PA1)
- net USART2_TX: now also JP9.1 (A)
- net ~CD: now also U1.CN3_9 (PB1), J4.1 (Pin_1); no longer U1.CN3_10 (PF0)
- net ~WP: now also U1.CN3_6 (PB0), J5.1 (Pin_1); no longer U1.CN3_11 (PF1)
- net AREF: now reaches U1.CN4_13 (AREF)
- net AREF: now also J10.1 (Pin_1)
- net PB0: no longer names the net of J23.1 (Pin_1)
- net PB0: now also J14.1 (Pin_1), JP2.2 (B); no longer U1.CN3_6 (PB0)
- net PB1: no longer names the net of J23.2 (Pin_2)
- net PB1: now also J15.1 (Pin_1), JP3.2 (B); no longer U1.CN3_9 (PB1)
- net PB2: no longer names the net of J23.3 (Pin_3)
- net PB2: now also J16.1 (Pin_1), JP4.2 (B)
- net PB5: no longer names the net of J23.6 (Pin_6)
- net PB5: now also J19.1 (Pin_1), JP7.2 (B); no longer U1.CN3_14 (PB5)
- net USAR2_RX renamed USART2_RX
- net USART2_RX: now also JP8.1 (A)
- new net: J17.1 (Pin_1), J23.4 (Pin_4), JP5.2 (B)
- new net: J18.1 (Pin_1), J23.5 (Pin_5), JP6.2 (B)
- new net: J20.1 (Pin_1), J23.7 (Pin_7), JP8.2 (B)
- new net: J21.1 (Pin_1), J23.8 (Pin_8), JP9.2 (B)
- new net PA0: JP4.1 (A), U1.CN4_12 (PA0)
- new net PA1: JP5.1 (A), U1.CN4_11 (PA1)
- new net PA3: JP6.1 (A), U1.CN4_10 (PA3)
- new net ~CS: J1.1 (DAT3/~CS), J6.1 (Pin_1), JP1.1 (A), R2.1
Other:
- note added: "1. SB16 and SB18 on F303 must be desoldered to enable SPI for pins PA5 and PA6"
- note added: "6. Kolla vad VREF ska vara på STM32 och CAN transceiver\n8. Kolla upp strömförsörjning, VIN/12V/5V/3V3. Varifrån kommer allt? \n9. Skaffa footprint till kondensatorer C1,C2"
- note added: "Links"
- note added: "NUCLEO32 - F303 / L432"
- note added: "Notes"
- note added: "Prospect SPI SD drivers"
- note added: "Right Screw Terminal and "breadboard""
- note added: "To Do"
- note added: "https://github.com/kiwih/cubemx-mmc-sd-card"
- note removed: "2. Se över vilka resistorvärden som behövs på 12-3.3V delarna"
- note removed: "5. Verifiera att VREF är kopplad till VDD på NUCLEO genom lödbrygga enligt datablad."
- note removed: "6. Kolla vad VREF ska vara på STM32 och CAN transceiver"
- note removed: "Anteckningar"
- note removed: "Onödig iom LDO på NUCLEO?"
- note removed: "Right Screw Terminal"
- note removed: "SD-kort drivers: https://github.com/kiwih/cubemx-mmc-sd-card"
- moved on the sheet: H1, H2, H3, H4, J1, J23, J24, R1, R10, R11, R12, R13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

Commit message: Vidareutveckling
Parts:
- removed J10, J14, J15, J16, J17, J18, J19, J20, J21, J22: Jumper, Vera-MRS-21:THT_Jumper, symbol Connector:Conn_01x01_Female
- added J13: Conn_01x11, Connector_PinHeader_2.54mm:PinHeader_1x11_P2.54mm_Vertical, symbol Connector_Generic:Conn_01x11
- renumbered J11 to J10, J12 to J11, J13 to J12, J23 to J14, J24 to J15
Connections:
- net +5V: now also J13.1 (Pin_1)
- net AREF: now also J13.3 (Pin_3)
- net GND: now also J13.2 (Pin_2)
- net at J14.1 (Pin_1), JP2.2 (B): now also J13.4 (Pin_4)
- net at J14.2 (Pin_2), JP3.2 (B): now also J13.5 (Pin_5)
- net at J14.3 (Pin_3), JP4.2 (B): now also J13.6 (Pin_6)
- net at J14.4 (Pin_4), JP5.2 (B): now also J13.7 (Pin_7)
- net at J14.5 (Pin_5), JP6.2 (B): now also J13.8 (Pin_8)
- net at J14.6 (Pin_6), JP7.2 (B): now also J13.9 (Pin_9)
- net at J14.7 (Pin_7), JP8.2 (B): now also J13.10 (Pin_10)
- net at J14.8 (Pin_8), JP9.2 (B): now also J13.11 (Pin_11)
- no-connect marks 0 -> 1
Other:
- note added: "8. Kolla upp strömförsörjning, VIN/12V/5V/3V3. Varifrån kommer allt? \n9. Skaffa footprint till kondensatorer C1,C2"
- note added: "Bottom Screw Terminal and header"
- note removed: "1. SB16 and SB18 on F303 must be desoldered to enable SPI for pins PA5 and PA6"
- note removed: "6. Kolla vad VREF ska vara på STM32 och CAN transceiver\n8. Kolla upp strömförsörjning, VIN/12V/5V/3V3. Varifrån kommer allt? \n9. Skaffa footprint till kondensatorer C1,C2"
- note removed: "Links"
- note removed: "Notes"
- note removed: "Prospect SPI SD drivers"
- note removed: "Right Screw Terminal and "breadboard""
- note removed: "To Do"
- note removed: "https://github.com/kiwih/cubemx-mmc-sd-card"
- moved on the sheet: C1, C2, J10, J11, J12, J14, J15, JP1, JP2, JP3, JP4, JP5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
