File: Motorrumsstyrning.sch (KiCad schematic (older format))
At the start: 51 parts, among them J1 SD_Card_Connector, J10 Jumper, J11 Jumper, J12 Jumper, J13 Conn_01x11, J14 Screw_Terminal_01x10, J15 Screw_Terminal_01x10, J2 Jumper, J3 Jumper, J4 Jumper, J5 Jumper, J6 Jumper, J7 Jumper, J8 Jumper, J9 Jumper, Q1 BC337, Q2 BC337, U1 NUCLEO-F303K8, U2 LM1084-5.0, U3 MCP2551-I-P

Commit message: Removed old code, generated new for F303K8
Parts:
- removed JP2, JP3: SolderJumper_2_Bridged, Jumper:SolderJumper-2_P1.3mm_Bridged2Bar_RoundedPad1.0x1.5mm, symbol Jumper:SolderJumper_2_Bridged
- J13: value Conn_01x11 -> Conn_01x09; footprint Connector_PinHeader_2.54mm:PinHeader_1x11_P2.54mm_Vertical -> Connector_PinHeader_2.54mm:PinHeader_1x09_P2.54mm_Vertical; symbol Connector_Generic:Conn_01x11 -> Connector_Generic:Conn_01x09
Connections:
- net PA8 is gone; now on net Tachometer: U1.CN3_12 (PA8)
- net +5V: now also J13.2 (Pin_2), J14.1 (Pin_1); no longer J13.1 (Pin_1)
- net AREF: now also J13.1 (Pin_1); no longer J13.3 (Pin_3)
- net Deadmans: now also U1.CN3_11 (PF1); no longer U1.CN3_10 (PF0)
- net GND: now also J13.3 (Pin_3), J14.2 (Pin_2); no longer J13.2 (Pin_2)
- net Injector_Enable: now also U1.CN4_9 (PA4); no longer U1.CN4_5 (PA2)
- net PA0: now also JP5.1 (A); no longer JP4.1 (A)
- net PA1: now also JP6.1 (A); no longer JP5.1 (A)
- net PA3: now also JP7.1 (A); no longer JP6.1 (A)
- net PB3: now also JP4.1 (A)
- net Start_Enable: no longer U1.CN3_14 (PB5)
- net Tachometer: no longer U1.CN3_11 (PF1)
- net at J13.4 (Pin_4): now also J14.3 (Pin_3), JP4.2 (B); no longer J14.1 (Pin_1)
- net at J13.5 (Pin_5): now also J14.4 (Pin_4), JP5.2 (B); no longer J14.2 (Pin_2)
- net at J14.5 (Pin_5), JP6.2 (B): now also J13.6 (Pin_6); no longer J13.8 (Pin_8)
- net at J14.6 (Pin_6), JP7.2 (B): now also J13.7 (Pin_7); no longer J13.9 (Pin_9)
- net at J14.7 (Pin_7), JP8.2 (B): now also J13.8 (Pin_8); no longer J13.10 (Pin_10)
- net at J14.8 (Pin_8), JP9.2 (B): now also J13.9 (Pin_9); no longer J13.11 (Pin_11)
- removed net PA4: JP7.1 (A), U1.CN4_9 (PA4)
- net USART2_RX renamed USART1_RX
- net USART2_TX renamed USART1_TX
- no-connect marks 1 -> 3
Other:
- note added: "8. Kolla upp strömförsörjning, VIN/12V/5V/3V3. kolla så källans max effek toch den förbrukade effekten stämmer överens.\n9. Skaffa footprint till kondensatorer C1,C2"
- note removed: "8. Kolla upp strömförsörjning, VIN/12V/5V/3V3. Varifrån kommer allt? \n9. Skaffa footprint till kondensatorer C1,C2"
Changed lines of the file:
@@
 $EndComp
 Text Label 7800 4200 0    50   ~ 0
-USART2_TX
+USART1_TX
 Text Label 7800 4300 0    50   ~ 0
-USART2_RX
+USART1_RX
 Text Label 6600 4000 2    50   ~ 0
 I2C1_SCL
@@
 Wire Notes Line
 	11150 4150 8750 4150
-Text Label 6600 4250 2    50   ~ 0
-Deadmans
-Text Label 6600 4350 2    50   ~ 0
+Text Label 6600 3700 2    50   ~ 0
+PB3
+Text Label 7800 4100 0    50   ~ 0
 Tachometer
 Wire Wire Line
@@
 	1    0    0    -1
 $EndComp
-$Comp
-L Motorrumsstyrning-rescue:Screw_Terminal_01x10-Connector J14
-U 1 1 60C79806
-P 10950 5250
-F 0 "J14" H 10900 5750 50  0000 L CNN
-F 1 "Screw_Terminal_01x10" V 11050 4800 50  0000 L CNN
-F 2 "Vera-MRS-21:TerminalBlock_Phoenix_MPT-0,5-10-2.54_1x10_P2.54mm_Horizontal" H 10950 5250 50  0001 C CNN
-F 3 "~" H 10950 5250 50  0001 C CNN
-	1    10950 5250
-	1    0    0    -1
-$EndComp
 Text Label 9450 5650 0    50   ~ 0
 Injector_IN
 Text Label 9450 5750 0    50   ~ 0
 Injector_OUT
-Text Label 6600 3900 2    50   ~ 0
+Text Label 6550 3900 2    50   ~ 0
 Start_Enable
 $Comp
@@
 Wire Wire Line
 	10150 1550 10850 1550
-Text Label 7800 3500 0    50   ~ 0
+Text Label 7800 3700 0    50   ~ 0
 Injector_Enable
 Text Label 9150 1750 0    50   ~ 0
@@
 Text Label 7800 3600 0    50   ~ 0
 PA3
-Text Label 6600 3700 2    50   ~ 0
-PB3
 Text Label 6600 3800 2    50   ~ 0
 PB4
-Text Label 7800 3700 0    50   ~ 0
-PA4
-Text Label 7800 4100 0    50   ~ 0
-PA8
-Text Label 9450 5050 0    50   ~ 0
+Text Label 6600 4350 2    50   ~ 0
+Deadmans
+Text Label 9450 5150 0    50   ~ 0
 PA0
-Text Label 9450 5150 0    50   ~ 0
+Text Label 9450 5250 0    50   ~ 0
 PA1
-Text Label 9450 5250 0    50   ~ 0
+Text Label 9450 5350 0    50   ~ 0
 PA3
-Text Label 9450 4850 0    50   ~ 0
-PB3
 Text Label 9450 5550 0    50   ~ 0
-USART2_TX
+USART1_TX
 Text Label 9450 5450 0    50   ~ 0
-USART2_RX
+USART1_RX
 $Comp
 L power:GND #PWR06
@@
 Wire Wire Line
 	6400 3150 6600 3150
-Wire Wire Line
-	6600 3150 6600 3100
-Wire Wire Line
-	6600 3150 6600 3200
-Connection ~ 6600 3150
 Text Label 10100 3100 0    50   ~ 0
 ~RST
@@
 L power:GND #PWR014
 U 1 1 60F3DE15
-P 10200 4450
-F 0 "#PWR014" H 10200 4200 50  0001 C CNN
-F 1 "GND" H 10200 4300 50  0000 C CNN
-F 2 "" H 10200 4450 50  0001 C CNN
-F 3 "" H 10200 4450 50  0001 C CNN
-	1    10200 4450
+P 9750 4800
+F 0 "#PWR014" H 9750 4550 50  0001 C CNN
+F 1 "GND" H 9750 4650 50  0000 C CNN
+F 2 "" H 9750 4800 50  0001 C CNN
+F 3 "" H 9750 4800 50  0001 C CNN
+	1    9750 4800
 	1    0    0    -1
 $EndComp
@@
 Wire Wire Line
 	3650 5800 4150 5800
-Text Label 9450 5350 0    50   ~ 0
-PA4
 Text Label 7800 3300 0    50   ~ 0
 PA0
@@
 Text Notes 8800 4250 0    50   ~ 0
 Bottom Screw Terminal and header
-$Comp
-L Jumper:SolderJumper_2_Bridged JP2
-U 1 1 612864F8
-P 10150 4850
-F 0 "JP2" H 9950 4900 50  0000 C CNN
-F 1 "SolderJumper_2_Bridged" H 10150 4964 50  0001 C CNN
-F 2 "Jumper:SolderJumper-2_P1.3mm_Bridged2Bar_RoundedPad1.0x1.5mm" H 10150 4850 50  0001 C CNN
-F 3 "~" H 10150 4850 50  0001 C CNN
-	1    10150 4850
-	1    0    0    -1
-$EndComp
-Wire Wire Line
-	9450 4850 10000 4850
-Wire Wire Line
-	9450 4950 10000 4950
 Wire Wire Line
 	9450 5050 10000 5050
@@
 Wire Wire Line
 	9450 5350 10000 5350
-$Comp
-L Jumper:SolderJumper_2_Bridged JP3
-U 1 1 61320BC4
-P 10150 4950
-F 0 "JP3" H 9950 5000 50  0000 C CNN
-F 1 "SolderJumper_2_Bridged" H 10150 5064 50  0001 C CNN
-F 2 "Jumper:SolderJumper-2_P1.3mm_Bridged2Bar_RoundedPad1.0x1.5mm" H 10150 4950 50  0001 C CNN
-F 3 "~" H 10150 4950 50  0001 C CNN
-	1    10150 4950
-	1    0    0    -1
-$EndComp
 $Comp
 L Jumper:SolderJumper_2_Bridged JP4
@@
 	1400 1400 1400 1300
 Connection ~ 1400 1400
-Text Label 9450 4950 0    50   ~ 0
-PA8
+Text Label 9450 5050 0    50   ~ 0
+PB3
 Wire Wire Line
 	8000 3150 7800 3150
@@
 L power:+5V #PWR016
 U 1 1 610F27A0
-P 10400 4550
-F 0 "#PWR016" H 10400 4400 50  0001 C CNN
-F 1 "+5V" H 10415 4723 50  0000 C CNN
-F 2 "" H 10400 4550 50  0001 C CNN
-F 3 "" H 10400 4550 50  0001 C CNN
-	1    10400 4550
+P 10000 4850
+F 0 "#PWR016" H 10000 4700 50  0001 C CNN
+F 1 "+5V" H 10000 5000 50  0000 C CNN
+F 2 "" H 10000 4850 50  0001 C CNN
+F 3 "" H 10000 4850 50  0001 C CNN
+	1    10000 4850
 	1    0    0    -1
 $EndComp
@@
 Wire Wire Line
 	10300 5050 10400 5050
-Wire Wire Line
-	10300 4950 10400 4950
-Wire Wire Line
-	10300 4850 10400 4850
-$Comp
-L Connector_Generic:Conn_01x11 J13
+$Comp
+L Connector_Generic:Conn_01x09 J13
 U 1 1 6114CA70
-P 10600 5050
-F 0 "J13" H 10500 5650 50  0000 L CNN
-F 1 "Conn_01x11" V 10700 5300 50  0000 L CNN
-F 2 "Connector_PinHeader_2.54mm:PinHeader_1x11_P2.54mm_Vertical" H 10600 5050 50  0001 C CNN
-F 3 "~" H 10600 5050 50  0001 C CNN
-	1    10600 5050
+P 10600 5150
+F 0 "J13" H 10500 5750 50  0000 L CNN
+F 1 "Conn_01x09" V 10700 5500 50  0000 L CNN
+F 2 "Connector_PinHeader_2.54mm:PinHeader_1x09_P2.54mm_Vertical" H 10600 5150 50  0001 C CNN
+F 3 "~" H 10600 5150 50  0001 C CNN
+	1    10600 5150
 	1    0    0    -1
 $EndComp
@@
 Wire Wire Line
 	10400 5550 10750 5550
-Connection ~ 10400 4850
-Wire Wire Line
-	10400 4850 10750 4850
-Connection ~ 10400 4950
-Wire Wire Line
-	10400 4950 10750 4950
 Connection ~ 10400 5050
 Wire Wire Line
@@
 	10200 4750 10400 4750
 Wire Wire Line
-	10200 4450 10300 4450
-Wire Wire Line
-	10300 4450 10300 4650
-Wire Wire Line
-	10300 4650 10400 4650
+	9750 4800 9900 4800
 NoConn ~ 6900 1600
 Text Notes 7000 6450 0    50   ~ 0
-8. Kolla upp strömförsörjning, VIN/12V/5V/3V3. Varifrån kommer allt? \n9. Skaffa footprint till kondensatorer C1,C2
+8. Kolla upp strömförsörjning, VIN/12V/5V/3V3. kolla så källans max effek toch den förbrukade effekten stämmer överens.\n9. Skaffa footprint till kondensatorer C1,C2
 Wire Notes Line
 	8750 4150 8750 5900
@@
 	1850 6150 3650 6150
 $Comp
-L Motorrumsstyrning-rescue:GND-power #PWR?
+L Motorrumsstyrning-rescue:GND-power #PWR0101
 U 1 1 6130AA47
 P 5800 4000
-F 0 "#PWR?" H 5800 3750 50  0001 C CNN
+F 0 "#PWR0101" H 5800 3750 50  0001 C CNN
 F 1 "GND" H 5805 3827 50  0000 C CNN
 F 2 "" H 5800 4000 50  0001 C CNN
@@
 	1    0    0    -1
 $EndComp
+NoConn ~ 7800 3500
+Wire Wire Line
+	6600 3100 6600 3150
+NoConn ~ 6600 4250
+Connection ~ 6600 3150
+Wire Wire Line
+	6600 3150 6600 3200
+$Comp
+L Motorrumsstyrning-rescue:Screw_Terminal_01x10-Connector J14
+U 1 1 60C79806
+P 10950 5250
+F 0 "J14" H 10900 5750 50  0000 L CNN
+F 1 "Screw_Terminal_01x10" V 11050 4800 50  0000 L CNN
+F 2 "Vera-MRS-21:TerminalBlock_Phoenix_MPT-0,5-10-2.54_1x10_P2.54mm_Horizontal" H 10950 5250 50  0001 C CNN
+F 3 "~" H 10950 5250 50  0001 C CNN
+	1    10950 5250
+	1    0    0    -1
+$EndComp
+Wire Wire Line
+	10750 4850 10400 4850
+Wire Wire Line
+	10400 4950 10750 4950
+Connection ~ 10400 4950
+Wire Wire Line
+	9900 4950 9900 4800
+Wire Wire Line
+	9900 4950 10400 4950
+Wire Wire Line
+	10000 4850 10400 4850
+Connection ~ 10400 4850
 $EndSCHEMATC
